File: GBA-Cartridge-Reader.kicad_sch (KiCad schematic)
At the start: 4 parts

Commit message: Schematic begun with various libraries. PCB design framework established.
Parts:
- removed U? (x2): 74LS595, symbol 74xx:74LS595
- removed U?: CartBus, symbol GBA:CartBus
- added C1, C2: 27PF-0603-50V-5%, Sparkfun-Capacitors:0603, symbol Capacitor-Sparkfun:27PF-0603-50V-5%
- added S1: MOMENTARY-SWITCH-SPST-2-SMD-4.6X2.8MM, Sparkfun-Switches:TACTILE_SWITCH_SMD_4.6X2.8MM, symbol SparkFun-Switches:MOMENTARY-SWITCH-SPST-2-SMD-4.6X2.8MM
- added XTAL1: C3E-16.000-9-1015-X-R, C3E-16.000-9-1015-X-R:C3E-16.000-9-1015-X-R, symbol 16MHz Clock:C3E-16.000-9-1015-X-R
- gave numbers to parts that had none: 1
Connections:
- net at U1.13 (~{RESET}): now also S1.1, S1.2
- net XTAL2: now reaches U1.16 (XTAL2)
- net XTAL2: now also C1.2, XTAL1.1
- net XTAL1: now reaches U1.17 (XTAL1)
- net XTAL1: now also C2.1, XTAL1.3
- new net GND: C1.1, C2.2, S1.3, S1.4, XTAL1.2, XTAL1.4

Commit message: Micro population complete.
Parts:
- added C10, C12, C3, C4: 0.1UF-0603-25V-5%, 0603, symbol Sparkfun-Capacitors:0.1UF-0603-25V-5%
- added C11: 1.0UF-0603-16V-10%, 0603, symbol Sparkfun-Capacitors:1.0UF-0603-16V-10%
- added CR1: CD1206-S01575, Arduino Diode:DIODE_CD1206-S01575_BRN, symbol Arduino Diode:CD1206-S01575
- added L1: MH2029-300Y, Arduino Buck:IND_BOURNS_MH2029, symbol Arduino Buck:MH2029-300Y
- added R1, R2: 22R, Resistor_SMD:R_0603_1608Metric, symbol Device:R_US
- added R5: 10K, Resistor_SMD:R_0603_1608Metric, symbol Device:R_US
Connections:
- net GND: now also U1.15 (GND), U1.23 (GND), U1.35 (GND), U1.43 (GND), U1.5 (UGND), C10.2, C11.2, C12.2, C3.1, C4.2
- net at S1.1, S1.2, U1.13 (~{RESET}): now also CR1., R5.2
- net +5V: now reaches U1.14 (VCC), U1.34 (VCC)
- net +5V: now also U1.2 (UVCC), C3.2, C4.1, CR1., L1.1, R5.1
- net at U1.24 (AVCC), U1.44 (AVCC): now also C12.1, L1.2
- net at U1.3 (D-): now also R1.1
- net at U1.4 (D+): now also R2.2
- net at U1.42 (AREF): now also C10.1
- net at U1.6 (UCAP): now also C11.1
- new net D+: R2.1
- new net D-: R1.2
Other:
- added sheet Power (GBA_Power.kicad_sch)
- moved on the sheet: S1
